File: pcb/qrp2350/qrp2350.kicad_sch (KiCad schematic)
At the start: 15 parts, among them J1 USB_C_Receptacle_USB2.0_14P, J2 Barrel_Jack, U1 RP2350B-QFN80, U2 NCP1117-3.3_SOT223, U3 LM7805_TO220

Commit message: update to start using full rpi pico 2
Parts:
- removed C1, C2, C3: 4.7u, Capacitor_SMD:C_0402_1005Metric, symbol Device:C
- removed C4, C5: 10u, symbol Device:C
- removed C6, C7: 0.33u, symbol Device:C
- removed D1: D, symbol Device:D
- removed J1: USB_C_Receptacle_USB2.0_14P, symbol Connector:USB_C_Receptacle_USB2.0_14P
- removed J2: Barrel_Jack, symbol Connector:Barrel_Jack
- removed L1: 3.3u, symbol Device:L
- removed R1: 33, Resistor_SMD:R_0402_1005Metric, symbol Device:R
- removed U1: RP2350B-QFN80, RP2350_KiCad-main:RP2350B_QFN-80_EP_10.573x10.573_Pitch0.4mm, symbol RP2350 QFN80:RP2350B-QFN80
- removed U2: NCP1117-3.3_SOT223, Package_TO_SOT_SMD:SOT-223-3_TabPin2, symbol Regulator_Linear:NCP1117-3.3_SOT223
- removed U3: LM7805_TO220, Package_TO_SOT_THT:TO-220-3_Vertical, symbol Regulator_Linear:LM7805_TO220
Connections:
- no-connect marks 1 -> 0

Commit message: 5/24/25
Parts:
- added A1: RaspberryPi_Pico, Module:RaspberryPi_Pico_Common_THT, symbol MCU_Module_RaspberryPi_Pico:RaspberryPi_Pico
- added C1: 100nF, symbol Device:C_Small_US
- added C10, C8: 220pF, symbol Device:C_Small
- added C11, C12: 0.1uF, symbol Device:C
- added C2: 5ohm, symbol Device:C_Small_US
- added C3, C4, C5, C6: 56nF, symbol Device:C_Small
- added C7, C9: 10uF, symbol Device:C_Small
- added J1: Conn_01x07_Pin, Connector_PinHeader_1.00mm:PinHeader_1x07_P1.00mm_Vertical, symbol Connector:Conn_01x07_Pin
- added J2: Conn_Coaxial, Connector_Coaxial:BNC_TEConnectivity_1478035_Horizontal, symbol Connector:Conn_Coaxial
- added Q1: BS170, Package_TO_SOT_THT:TO-92L_HandSolder, symbol Transistor_FET:BS170
- added R1: 0.056ohm, symbol Device:R_Small_US
- added R10, R9: 10k, symbol Device:R
- added R2: 1nF, symbol Device:R_Small_US
- added R3, R4, R6, R7: 82ohm, symbol Device:R_Small_US
- added R5, R8: 56kohm, symbol Device:R_Small_US
- added U1: 14529, Package_DIP:DIP-16_W7.62mm, symbol 4xxx:14529
- added U2: MCP6022, Package_DIP:DIP-8_W7.62mm, symbol Amplifier_Operational:MCP6022
Connections:
- new net: R4.1, U2.3 (+)
- new net: C6.1, R4.2, U1.5 (X3)
- new net: C10.1, R6.2, R8.1, U2.5 (+)
- new net: C1.1, C11.1, J2.1 (In), R10.1, R9.2
- new net: C5.1, C7.1, U1.2 (X0)
- new net: C8.1, R3.2, R5.1, U2.2 (-)
- new net: C3.1, C9.1, U1.3 (X1)
- new net: C9.2, R6.1
- new net: C4.1, R7.2, U1.4 (X2)
- new net: C1.2, R1.1, R2.1
- new net: R7.1, U2.6 (-)
- new net: C2.1, Q1.1 (D), R2.2
- new net: Q1.3 (S), U1.9 (Z)
- new net: C7.2, R3.1
- new net: C2.2, R1.2
- new net +3.3V: A1.36 (3V3), J1.1 (Pin_1), R9.1, U1.1 (STX), U1.15 (STY), U1.16 (VDD), U2.8 (V+)
- new net GND: A1.13 (GND), A1.18 (GND), A1.23 (GND), A1.28 (GND), A1.3 (GND), A1.33 (AGND), A1.38 (GND), A1.8 (GND), C11.2, C12.2, C3.2, C4.2, C5.2, C6.2, J1.2 (Pin_2), J2.2 (Ext), R10.2, U1.8 (VSS), U2.4 (V-)
- new net RX_I: A1.31 (GPIO26_ADC0), C10.2, R8.2, U2.7
- new net RX_Q: A1.32 (GPIO27_ADC1), C8.2, R5.2, U2.1
- new net SCL1: J1.4 (Pin_4)
- new net SDA1: J1.3 (Pin_3)
- new net TX_SW: C12.1, Q1.2 (G)
- new net XTAL_0: J1.7 (Pin_7), U1.6 (A)
- new net XTAL_1: J1.6 (Pin_6), U1.7 (B)
- new net XTAL_2: J1.5 (Pin_5)
- no-connect marks 0 -> 5
Other:
- note added: "Band Pass Filter for 28mHz-29.7mHz"

Commit message: created transmitter side stuff
Parts:
- removed C1: 100nF, symbol Device:C_Small_US
- removed C2: 5ohm, symbol Device:C_Small_US
- removed R1: 0.056ohm, symbol Device:R_Small_US
- removed R10, R9: 10k, symbol Device:R
- removed R2: 1nF, symbol Device:R_Small_US
- added C1: 0.1uF, symbol Device:C
- added C13: 100uF, symbol Device:C
- added C14: C, symbol Device:C
- added C15, C18: 56pF, symbol Device:C
- added C16, C17: 150pF, symbol Device:C
- added C2: 1nF, symbol Device:C
- added J3: AudioJack2_Ground_Switch, Connector_Audio:Jack_3.5mm_CUI_SJ1-3515N_Horizontal, symbol Connector_Audio:AudioJack2_Ground_Switch
- added L1: 0.28 uH, symbol Device:L_Iron
- added L2, L4: 303nH, symbol Device:L_Iron
- added L3: 382nH, symbol Device:L_Iron
- added Q2, Q3, Q4: BS170, Package_TO_SOT_THT:TO-92_Inline, symbol Transistor_FET:BS170
- added R11: 100ohm, symbol Device:R
- added U3: 7400, Package_DIP:DIP-14_W7.62mm, symbol 74xx:7400
Connections:
- net +3.3V: now also U3.14 (VCC)
- net GND: now also C1.1, C14.1, C15.2, C16.2, C17.2, C18.2, J3.G, Q2.3 (S), Q3.3 (S), Q4.3 (S), U3.7 (GND); no longer C11.2
- net XTAL_2: now also U3.1, U3.10
- net at J2.1 (In): now also C18.1, L4.2; no longer C11.1
- net Speaker: now reaches A1.21 (GPIO16)
- net Speaker: now also C13.1
- net at Q1.1 (D): now also C2.1
- net RF_IN: now reaches Q1.3 (S), U1.9 (Z)
- new net: C13.2, R11.1
- new net: C14.2, J3.S, J3.T, R11.2
- new net: C17.1, L3.2, L4.1
- new net: C11.2, C15.1, L2.1
- new net: C16.1, L2.2, L3.1
- new net: C11.1, C2.2, L1.2, Q2.1 (D), Q3.1 (D), Q4.1 (D)
- new net: Q2.2 (G), Q3.2 (G), Q4.2 (G), U3.6
- new net: U3.4, U3.5, U3.8
- new net: C1.2, L1.1
- new net RX: U3.12, U3.13
- new net TX: U3.11, U3.9
Other:
- note added: "Low Pass Filter for 28mHz-29.7mHz"
- note removed: "Band Pass Filter for 28mHz-29.7mHz"
- moved on the sheet: C10, C12, C3, C4, C5, C6, C7, C8, C9, J2, Q1, R3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

Commit message: AHHHH
Parts:
- added J4: Barrel_Jack, Connector_BarrelJack:BarrelJack_SwitchcraftConxall_RAPC10U_Horizontal, symbol Connector:Barrel_Jack
Connections:
- net KEY_OUT: now reaches A1.22 (GPIO17)
Changed lines of the file:
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@@
+		)
+	)
+	(global_label "KEY_OUT"
+		(shape input)
+		(at 83.82 97.79 0)
+		(fields_autoplaced yes)
+		(effects
+			(font
+				(size 1.27 1.27)
+			)
+			(justify left)
+		)
+		(property "Intersheetrefs" "${INTERSHEET_REFS}"
+			(at 94.909 97.79 0)
+			(effects
+				(font
+					(size 1.27 1.27)
+				)
+				(justify left)
+				(hide yes)
+			)
 		)
 	)
@@
 					(unit 1)
 				)
+			)
+		)
+	)
+	(symbol
+		(lib_id "Connector:Barrel_Jack")
+		(at 116.84 182.88 0)
+		(unit 1)
+		(exclude_from_sim no)
+		(in_bom yes)
+		(on_board yes)
+		(dnp no)
+		(fields_autoplaced yes)
+		(property "Reference" "J4"
+			(at 116.84 173.99 0)
+			(effects
+				(font
+					(size 1.27 1.27)
+				)
+			)
+		)
+		(property "Value" "Barrel_Jack"
+			(at 116.84 176.53 0)
+			(effects
+				(font
+					(size 1.27 1.27)
+				)
+			)
+		)
+		(property "Footprint" "Connector_BarrelJack:BarrelJack_SwitchcraftConxall_RAPC10U_Horizontal"
+			(at 118.11 183.896 0)
+			(effects
+				(font
+					(size 1.27 1.27)
+				)
+				(hide yes)
+			)
+		)
+		(property "Datasheet" "~"
+			(at 118.11 183.896 0)
+			(effects
+				(font
+					(size 1.27 1.27)
+				)
+				(hide yes)
+			)
+		)
+		(property "Description" "DC Barrel Jack"
+			(at 116.84 182.88 0)
+			(effects
+				(font
+					(size 1.27 1.27)
+				)
+				(hide yes)
+			)
+		)
+		(pin "2"
+		)
+		(pin "1"
+		)
+		(instances
+			(project ""
+				(path "/6fac9320-a328-4a81-9076-6d5cad0da2c8"
+					(reference "J4")
+					(unit 1)
+				)
